Commit message: Create gpu to enable/disable GPU processing

File: ca_description/urdf/create_2.urdf.xacro (robot description, xacro)
@@ -7,4 +7,4 @@
   </xacro:create_base>
   <!-- Roomblock -->
-  <xacro:roomblock parent="base_link" visualize="$(arg visualize)"/>
+  <xacro:roomblock parent="base_link" visualize="$(arg visualize)" gpu="$(arg gpu)"/>
 </robot>

File: ca_description/urdf/roomblock.urdf.xacro (robot description, xacro)
@@ -8,5 +8,5 @@
   <xacro:include filename="$(find ca_description)/urdf/sensors/laser_sensor.xacro"/>
   <xacro:include filename="$(find ca_description)/urdf/sensors/camera_sensor.xacro"/>
-  <xacro:macro name="roomblock" params="parent visualize:=false">
+  <xacro:macro name="roomblock" params="parent visualize:=false gpu:=false">
     <xacro:property name="z" value="0.061"/>
     <xacro:property name="roomblock_link" value="block_link"/>
@@ -25,5 +25,5 @@
       </visual>
     </link>
-    <xacro:laser_sensor parent="${roomblock_link}" visualize="$(arg visualize)"/>
+    <xacro:laser_sensor parent="${roomblock_link}" visualize="${visualize}" gpu="${gpu}"/>
     <xacro:camera_sensor parent="${roomblock_link}"/>
     <xacro:roomblock_gazebo link_name="${roomblock_link}"/>
