Commit message: Fix URDF to include contact in bumpers

File: ca_description/urdf/create_base.urdf.xacro (robot description, xacro)
@@ -9,18 +9,16 @@
     <xacro:include filename="$(find ca_description)/urdf/sensors/cliff_sensors.xacro"/>
     <link name="base_footprint">
-    <visual>
-      <origin xyz="0 0 0" rpy="0 0 0" />
-      <geometry>
-        <box size="0.001 0.001 0.001" />
-      </geometry>
-      <material name="Green" />
-    </visual>
-    <collision>
+      <collision name="base_footprint">
+        <origin xyz="0.0 0.0 0.0308" rpy="0 0 0" />
+        <geometry>
+          <cylinder length="0.0611632" radius="0.16495" />
+        </geometry>
+      </collision>
+    </link>
+    <joint name="base_joint" type="fixed">
       <origin xyz="0 0 0.017" rpy="0 0 0" />
-      <geometry>
-        <box size="0.001 0.001 0.001" />
-      </geometry>
-    </collision>
-    </link>
+      <parent link="base_footprint" />
+      <child link="base_link" />
+    </joint>
     <link name="base_link">
       <inertial>
@@ -35,5 +33,5 @@
         </geometry>
       </visual>
-      <collision>
+      <collision name="base_link">
         <origin xyz="0.0 0.0 0.0308" rpy="0 0 0" />
         <geometry>
@@ -42,9 +40,4 @@
       </collision>
     </link>
-    <joint name="base_footprint_joint" type="fixed">
-      <origin xyz="0 0 0.017" rpy="0 0 0" />
-      <parent link="base_footprint" />
-      <child link="base_link" />
-    </joint>
     <xacro:wall_sensor visualize="${visualize}"/>
     <xacro:cliff_sensors visualize="${visualize}"/>

File: ca_description/urdf/create_base_gazebo.urdf.xacro (robot description, xacro)
@@ -38,5 +38,5 @@
     </gazebo>
     <!-- Bumpers -->
-    <gazebo reference="base_link">
+    <gazebo reference="base_footprint">
       <gravity>true</gravity>
       <self_collide>false</self_collide>
@@ -45,10 +45,9 @@
         <update_rate>50</update_rate>
         <contact>
-          <collision>base_link_collision</collision>
-          <topic>bumpers</topic>
+          <collision>base_footprint_collision</collision>
         </contact>
         <!-- Plugin -->
         <plugin name="create_bumper_controller" filename="libcreate_bumper_plugin.so">
-          <frameName>base_link</frameName>
+          <frameName>base_footprint</frameName>
           <bumperTopicName>bumper</bumperTopicName>
         </plugin>

Commit message: Add GPU flag

File: ca_description/urdf/create_base.urdf.xacro (robot description, xacro)
@@ -1,5 +1,5 @@
 <?xml version="1.0" ?>
 <robot xmlns:xacro="http://ros.org/wiki/xacro">
-  <xacro:macro name="create_base" params="diffdrive_update_rate:=40 wheel_separation wheel_radius:=0.036 wheel_width:=0.024 wheel_torque:=0.5 wheel_accel:=0.5 mass_kg:=3.5 base_diameter *mesh visualize:=false">
+  <xacro:macro name="create_base" params="diffdrive_update_rate:=40 wheel_separation wheel_radius:=0.036 wheel_width:=0.024 wheel_torque:=0.5 wheel_accel:=0.5 mass_kg:=3.5 base_diameter *mesh visualize:=false gpu:=false">
     <xacro:include filename="$(find ca_description)/urdf/create_base_gazebo.urdf.xacro"/>
     <xacro:include filename="$(find ca_description)/urdf/create_caster_wheel.xacro"/>
@@ -47,6 +47,6 @@
       <child link="base_link" />
     </joint>
-    <xacro:wall_sensor visualize="${visualize}"/>
-    <xacro:cliff_sensors visualize="${visualize}"/>
+    <xacro:wall_sensor visualize="${visualize}" gpu="${gpu}"/>
+    <xacro:cliff_sensors visualize="${visualize}" gpu="${gpu}"/>
     <xacro:imu_sensor/>
     <xacro:create_wheel prefix="left" y_offset="${wheel_separation / 2}" wheel_radius="${wheel_radius}" wheel_width="${wheel_width}"/>

File: ca_description/urdf/sensors/camera_sensor_gazebo.xacro (robot description, xacro)
@@ -7,5 +7,5 @@
       <update_rate>30.0</update_rate>
       <camera name="head">
-        <horizontal_fov>1.3962634</horizontal_fov>
+        <horizontal_fov>${80*pi/180.}</horizontal_fov>
         <image>
           <width>800</width>
