Commit message: ¨Code¨

File: ca_description/urdf/create_base.xacro (robot description, xacro)
@@ -8,4 +8,5 @@
     <xacro:include filename="$(find ca_description)/urdf/sensors/wall_sensor.xacro"/>
     <xacro:include filename="$(find ca_description)/urdf/sensors/cliff_sensors.xacro"/>
+    <xacro:include filename="$(find ca_description)/urdf/sensors/internal_imu_angle.xacro"/>
     <xacro:property name="base_link_offset_z" value="0.0308"/>
     <xacro:property name="base_offset_z" value="0.017"/>
@@ -35,5 +36,7 @@
     <xacro:wall_sensor visualize="${visualize}"/>
     <xacro:cliff_sensors visualize="${visualize}"/>
-    <xacro:imu_sensor/>
+    <xacro:imu_sensor name="imu">
+      <origin xyz="0 -0.04 0.13" rpy="0 0 0"/>
+    </xacro:imu_sensor>
     <xacro:create_wheel prefix="left" y_offset="${wheel_separation / 2}" wheel_radius="${wheel_radius}" wheel_width="${wheel_width}"/>
     <xacro:create_wheel prefix="right" y_offset="${wheel_separation / -2}" wheel_radius="${wheel_radius}" wheel_width="${wheel_width}"/>

Commit message: Internal imu code, xacro and cpp

File: ca_description/urdf/create_base.xacro (robot description, xacro)
@@ -36,7 +36,7 @@
     <xacro:wall_sensor visualize="${visualize}"/>
     <xacro:cliff_sensors visualize="${visualize}"/>
-    <xacro:imu_sensor name="imu">
-      <origin xyz="0 -0.04 0.13" rpy="0 0 0"/>
-    </xacro:imu_sensor>
+    <xacro:internal_imu_angle name="internal_imu_angle">
+      <origin xyz="0 0 0" rpy="0 0 0"/>
+    </xacro:internal_imu_angle>
     <xacro:create_wheel prefix="left" y_offset="${wheel_separation / 2}" wheel_radius="${wheel_radius}" wheel_width="${wheel_width}"/>
     <xacro:create_wheel prefix="right" y_offset="${wheel_separation / -2}" wheel_radius="${wheel_radius}" wheel_width="${wheel_width}"/>

File: ca_description/urdf/roomblock.xacro (robot description, xacro)
@@ -38,4 +38,7 @@
     <xacro:camera_sensor parent="${roomblock_link}"/>
     <xacro:roomblock_gazebo link_name="${roomblock_link}"/>
+    <xacro:imu_sensor name="imu">
+      <origin xyz="0 -0.04 0.13" rpy="0 0 0"/>
+    </xacro:imu_sensor>
   </xacro:macro>
 </robot>

File: ca_description/urdf/sensors/internal_imu_angle.xacro (robot description, xacro)
@@ -1,5 +1,5 @@
 <?xml version="1.0" ?>
 <robot xmlns:xacro="http://ros.org/wiki/xacro">
-<xacro:macro name="internal_imu" params="name *origin">
+<xacro:macro name="internal_imu_angle" params="name *origin">
   <xacro:include filename="$(find ca_description)/urdf/common_properties.xacro"/>
   <xacro:include filename="$(find ca_description)/urdf/sensors/internal_imu_angle_gazebo.xacro"/>
@@ -14,5 +14,5 @@
     <xacro:dummy_inertia/>
   </link>
-  <xacro:internal_imu_angle_gazebo link_name="${link_name}"/>
+  <xacro:internal_imu_angle_gazebo name="internal_imu_angle" link_name="${link_name}"/>
 </xacro:macro>
 </robot>

File: ca_description/urdf/sensors/internal_imu_angle_gazebo.xacro (robot description, xacro)
@@ -3,11 +3,11 @@
 <xacro:macro name="internal_imu_angle_gazebo" params="name link_name">
   <gazebo>
-    <plugin name="internal_imu_angle_controller" filename="libgazebo_ros_internal_imu.so">
+    <plugin name="internal_imu_angle_controller" filename="/home/tomas/catkin_ws/src/create_autonomy/ca_gazebo/devel/lib/libgazebo_ros_internal_imu.so">
       <alwaysOn>true</alwaysOn>
       <updateRate>30</updateRate>
       <bodyName>${link_name}</bodyName>
-      <topicName>${name}/data</topicName>
-      <serviceName>${name}/is_calibrated</serviceName>
-      <gaussianNoise>${0.0017*0.0017}</gaussianNoise>
+      <topicName>${name}</topicName>
+      <serviceName>${name}</serviceName>
+      <gaussianNoise>${0.1*0.1}</gaussianNoise>
       <xyzOffsets>0 0 0</xyzOffsets>
       <rpyOffsets>0 0 0</rpyOffsets>
